File: nRF54L15_nPM2100_CR2032.kicad_pcb (KiCad board)
At the start: 4 copper layers, 32 x 28.7 mm, 29 parts, among them SW1 SW_Push, U1 nRF54L15-CAXX, U2 nPM2100-CAXX, Y1 32.768kHz, Y2 SiT11100

Commit message: Routing complete
Parts:
- removed REF** (x2): PinHeader_1x04_P2.54mm_Vertical, Connector_PinHeader_2.54mm:PinHeader_1x04_P2.54mm_Vertical
- added J1: Conn_ARM_SWD_TagConnect_TC2030-NL, Connector:Tag-Connect_TC2030-IDC-NL_2x03_P1.27mm_Vertical, F.Cu at (197.2, 59.4)
- added JP1: Jumper_2_Small_Bridged, Jumper:SolderJumper-2_P1.3mm_Bridged_RoundedPad1.0x1.5mm, F.Cu at (180.4, 58.4)
- added Q1: Q_NMOS_GSD, Package_TO_SOT_SMD:SOT-23, F.Cu at (184.6, 51.0)
- added R1: 350R, Resistor_SMD:R_0402_1005Metric, F.Cu at (187.0, 50.5)
- added R2: 10kR, Resistor_SMD:R_0201_0603Metric, F.Cu at (183.9, 58.2)
- added R3: 10kR, Resistor_SMD:R_0201_0603Metric, F.Cu at (184.6, 58.2)
- added R4: 1MR, Resistor_SMD:R_0402_1005Metric, F.Cu at (182.1, 51.0)
- added TP1: TestPoint, TestPoint:TestPoint_Pad_D1.0mm, F.Cu at (195.0, 55.0)
- added TP2: TestPoint, TestPoint:TestPoint_Pad_D1.0mm, F.Cu at (197.0, 55.0)
- AE1: footprint RF_Antenna:Johanson_2450AT18x100 -> hlord2000-RF_Antenna:Ignion_NN02-101
- C6, C9: footprint Capacitor_SMD:C_0201_0603Metric -> Capacitor_SMD:C_01005_0402Metric
- D1: value LED_Small -> APT3216LVBC/D; footprint LED_SMD:LED_0603_1608Metric -> LED_SMD:LED_1206_3216Metric
- L2, L3, L4: footprint Capacitor_SMD:C_0201_0603Metric -> Inductor_SMD:L_01005_0402Metric
- moved D1 13.0 mm to (190.0, 50.0), turned to 0 degrees
- moved SW1 7.99 mm to (190.0, 55.0), turned to 0 degrees
- moved L5 6.90 mm to (184.7, 61.9), turned to 0 degrees
- moved C3 6.39 mm to (186.0, 62.1), turned to 90 degrees
- moved C13 4.87 mm to (186.9, 61.2), turned to -90 degrees
- moved U2 4.55 mm to (185.1, 60.1), turned to -90 degrees
- moved C4 2.61 mm to (185.6, 58.5), turned to 180 degrees
- moved C7 2.58 mm to (186.8, 59.5), turned to 90 degrees
- moved Y1 1.73 mm to (191.8, 58.4)
- moved C1 1.09 mm to (189.1, 60.0)
- moved C10 1.09 mm to (190.2, 58.1)
- moved C11 1.09 mm to (190.2, 58.8)
- moved C12 1.09 mm to (188.4, 61.4)
- moved C2 1.09 mm to (187.7, 61.4)
- moved C5 1.09 mm to (189.1, 61.4)
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Connections:
- AE1 pad 1: GND -> unconnected-(AE1-FEED-Pad1)
- C3 pad 1: Net-(BT1-+) -> Net-(JP1-B)
- L5 pad 1: Net-(BT1-+) -> Net-(JP1-B)
- SW1 pad 1: unconnected-(SW1-Pad1) -> Net-(U2-SHPHLD)
- SW1 pad 2: unconnected-(SW1-Pad2) -> GND
- U1 pad B3: unconnected-(U1-P1.09-PadB3) -> /LED
- U1 pad D2: unconnected-(U1-~{RESET}-PadD2) -> Net-(J1-~{RESET})
- U1 pad D5: unconnected-(U1-P1.03-PadD5) -> /SCL
- U1 pad D6: unconnected-(U1-P1.04-PadD6) -> /SDA
- U1 pad E3: unconnected-(U1-SWDCLK-PadE3) -> Net-(J1-SWCLK)
- U1 pad E7: unconnected-(U1-P1.07-PadE7) -> /UART_TX
- U1 pad F2: unconnected-(U1-SWDIO-PadF2) -> Net-(J1-SWDIO)
- U1 pad F7: unconnected-(U1-P1.08-PadF7) -> /UART_RX
- U2 pad C2: unconnected-(U2-SYSGDEN-PadC2) -> GND
- U2 pad C4: Net-(BT1-+) -> Net-(JP1-B)
- U2 pad D2: unconnected-(U2-SCL-PadD2) -> /SCL
- U2 pad D3: unconnected-(U2-SDA-PadD3) -> /SDA
- U2 pad D4: unconnected-(U2-SHPHLD-PadD4) -> Net-(U2-SHPHLD)
Routing:
- net VDD: track 0.00 -> 35.1 mm, vias 0 -> 7
- net /LED: track 0.00 -> 20.9 mm, vias 0 -> 2
- net Net-(U2-SHPHLD): track 0.00 -> 17.2 mm
- net Net-(J1-SWCLK): track 0.00 -> 11.9 mm, vias 0 -> 2
- net Net-(J1-SWDIO): track 0.00 -> 11.8 mm, vias 0 -> 2
- net /SDA: track 0.00 -> 10.5 mm, vias 0 -> 2
- net GND: track 0.00 -> 10.2 mm, vias 0 -> 24
- net /SCL: track 0.00 -> 10.0 mm, vias 0 -> 2
- net Net-(J1-~{RESET}): track 0.00 -> 9.09 mm, vias 0 -> 2
- net Net-(JP1-B): track 0.00 -> 8.94 mm
- net /UART_RX: track 0.00 -> 7.80 mm, vias 0 -> 2
- net /UART_TX: track 0.00 -> 7.11 mm, vias 0 -> 2
- net Net-(U1-DECA): track 0.00 -> 5.27 mm, vias 0 -> 2
- net Net-(BT1-+): track 0.00 -> 4.16 mm, vias 0 -> 1
- net Net-(AE1-PCB_Trace): track 0.00 -> 3.91 mm
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- added copper zone on In1.Cu, net GND
- added copper zone on In2.Cu, net GND
Other:
- board text removed: "2100"
- board text removed: "54L15"
- board text removed: "SWD"
- board text removed: "SiT11100"

Commit message: Nov. 7th 2024
Parts:
- added C14: 1nF, Capacitor_SMD:C_0201_0603Metric, F.Cu at (187.1, 62.4)
- added C15: 0.22uF, Capacitor_SMD:C_0201_0603Metric, F.Cu at (196.4, 49.0)
- added C16: 100nF, Capacitor_SMD:C_0201_0603Metric, F.Cu at (195.4, 47.9)
- added C17: 100nF, Capacitor_SMD:C_0201_0603Metric, F.Cu at (193.3, 49.1)
- added C18: NA, Capacitor_SMD:C_0201_0603Metric, F.Cu at (189.4, 67.0)
- added C19: 2.2uF, Capacitor_SMD:C_0201_0603Metric, F.Cu at (185.6, 58.5)
- added C20: 2.2uF, Capacitor_SMD:C_0201_0603Metric, F.Cu at (185.9, 48.1)
- added JP2: Jumper_3_Open, Jumper:SolderJumper-3_P1.3mm_Open_RoundedPad1.0x1.5mm, F.Cu at (176.4, 56.6)
- added JP3: Jumper_2_Small_Bridged, Jumper:SolderJumper-2_P1.3mm_Bridged_RoundedPad1.0x1.5mm, F.Cu at (177.8, 53.7)
- added JP4: Jumper_2_Small_Bridged, Jumper:SolderJumper-2_P1.3mm_Bridged_RoundedPad1.0x1.5mm, F.Cu at (180.3, 53.7)
- added L6: NA, Inductor_SMD:L_0201_0603Metric, F.Cu at (190.5, 67.4)
- added L7: NA, Inductor_SMD:L_0201_0603Metric, F.Cu at (188.4, 67.4)
- added MK1: MP34DT05-A, hlord2000-Sensor_Audio:ST_HCLGA-4_3x4mm_P1.35mm, F.Cu at (184.0, 50.0)
- added U3: ADXL366, hlord2000-Sensor_Motion:Analog_LGA-12_2.20x2.30mm_P0.5mm, F.Cu at (195.0, 50.0)
- C10, C3: footprint Capacitor_SMD:C_0201_0603Metric -> Capacitor_SMD:C_0402_1005Metric
- C13: value 22uF -> 10uF
- C4: value 2.2uF -> 1nF
- C6, C9: footprint Capacitor_SMD:C_01005_0402Metric -> Capacitor_SMD:C_0201_0603Metric
- L2, L3, L4: footprint Inductor_SMD:L_01005_0402Metric -> Inductor_SMD:L_0201_0603Metric
- Q1: footprint Package_TO_SOT_SMD:SOT-23 -> Package_DFN_QFN:Diodes_DFN1006-3
- moved JP1 6.97 mm to (175.3, 53.7), turned to -90 degrees
- moved R4 3.04 mm to (184.1, 53.3), turned to 180 degrees
- moved C4 2.44 mm to (187.8, 59.6), turned to 0 degrees
- moved Q1 1.60 mm to (185.8, 52.0), turned to 90 degrees
- moved AE1 1.50 mm to (188.8, 69.8), turned to 180 degrees
- moved R1 1.49 mm to (187.0, 52.0)
- moved C10 0.38 mm to (189.9, 57.8)
- moved C3 0.20 mm to (185.9, 62.3)
- moved L5 0.19 mm to (184.5, 61.9)
- moved C8 0.12 mm to (192.4, 60.7)
Connections:
- net Net-(BT1-+) renamed VBAT
- C4 pad 1: Net-(U2-VOUTLDO) -> Net-(U2-VINT)
- C7 pad 1: VDD -> Net-(JP3-A)
- L4 pad 2: Net-(AE1-PCB_Trace) -> Net-(L4-Pad2)
- SW1 pad 1: Net-(U2-SHPHLD) -> /BUTTON0
- U1 pad B6: unconnected-(U1-P1.15-PadB6) -> /BUTTON0
- U1 pad C3: unconnected-(U1-P1.10-PadC3) -> /GPIO0
- U1 pad E1: unconnected-(U1-P0.03-PadE1) -> /PDM_CLK
- U1 pad F1: unconnected-(U1-P0.01-PadF1) -> /PDM_DATA
- U1 pad G1: unconnected-(U1-P0.00-PadG1) -> /INT1
- U2 pad A1: Net-(U2-VOUTLDO) -> Net-(JP4-A)
- U2 pad A2: VDD -> Net-(JP3-A)
- U2 pad C3: unconnected-(U2-GPIO0-PadC3) -> /GPIO0
- U2 pad D4: Net-(U2-SHPHLD) -> /BUTTON0
Routing:
- net /VDD_LDO: track 0.00 -> 40.5 mm, vias 0 -> 4
- net /BUTTON0: track 0.00 -> 24.2 mm, vias 0 -> 2
- net /PDM_CLK: track 0.00 -> 22.6 mm, vias 0 -> 2
- net /PDM_DATA: track 0.00 -> 21.6 mm, vias 0 -> 2
- net /SCL: track 10.0 -> 29.3 mm, vias 2 -> 3
- net Net-(U2-SHPHLD): track 17.2 -> 0.00 mm
- net /SDA: track 10.5 -> 27.4 mm, vias 2 -> 3
- net Net-(JP3-A): track 0.00 -> 15.9 mm, vias 0 -> 2
- net /INT1: track 0.00 -> 14.2 mm
- net VDD: track 35.1 -> 46.9 mm
- net Net-(JP4-A): track 0.00 -> 10.3 mm, vias 0 -> 2
- net Net-(JP1-B): track 8.94 -> 19.1 mm, vias 0 -> 2
- net /GPIO0: track 0.00 -> 5.90 mm, vias 0 -> 2
- net VBAT: track 4.16 -> 0.00 mm, vias 1 -> 2
- net /LED: track 20.9 -> 17.3 mm
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Other:
- board text added: "LAYER 1 - 1 OZ COPPER - (0.0175 MM) LAYER 2 - PREPREG (7628, DK 4.74, 0.1855 MM) LAYER 3 - 1 OZ COPPER - (0.0350 MM) LAYER 4 - CORE (DK 4.6, 1.03 MM) LAYER 5 - 1 OZ COPPER - (0.0350 MM) LAYER 6 - PREPREG (7628, DK 4.74, 0.1855 MM) LAYER 7 - 1 OZ COPPER - (0.0175 MM)"
- board text removed: "UART"

Commit message: Dec92024
Parts:
- removed C13: 10uF, Capacitor_SMD:C_0402_1005Metric
- removed C14: 1nF, Capacitor_SMD:C_0201_0603Metric
- removed C18: NA, Capacitor_SMD:C_0201_0603Metric
- removed C19, C7: 2.2uF, Capacitor_SMD:C_0201_0603Metric
- removed JP4: Jumper_2_Small_Bridged, Jumper:SolderJumper-2_P1.3mm_Bridged_RoundedPad1.0x1.5mm
- removed L5: 2.2uH, Inductor_SMD:L_0402_1005Metric
- added L18: 4.7nH, Capacitor_SMD:C_0201_0603Metric, F.Cu at (189.4, 67.0)
- C3: value 10uF -> 100nF; footprint Capacitor_SMD:C_0402_1005Metric -> Capacitor_SMD:C_0201_0603Metric
- C4: value 1nF -> 100nF
- JP2: value Jumper_3_Open -> Jumper_2_Small_Bridged; footprint Jumper:SolderJumper-3_P1.3mm_Open_RoundedPad1.0x1.5mm -> Resistor_SMD:R_0402_1005Metric
- JP3: footprint Jumper:SolderJumper-2_P1.3mm_Bridged_RoundedPad1.0x1.5mm -> Resistor_SMD:R_0402_1005Metric
- L3: value 4.6nH -> 4.7nH
- L6: value NA -> 4.7nH; footprint Inductor_SMD:L_0201_0603Metric -> Capacitor_SMD:C_0201_0603Metric
- L7: value NA -> 10nH; footprint Inductor_SMD:L_0201_0603Metric -> Capacitor_SMD:C_0201_0603Metric
- R1: value 350R -> 1kR
- U1: footprint nordic-lib-kicad-nrf54:BGA-49_7x7_2.3984x2.2309mm -> nordic-lib-kicad-nrf54:BGA-47_7x7_2.451x2.245mm
- U2: value nPM2100-CAXX -> SiP32432DR3; footprint nordic-lib-kicad-npm:BGA-16_4x4_1.9175x1.8975mm -> Package_TO_SOT_SMD:SOT-363_SC-70-6
- moved JP2 19.2 mm to (193.3, 47.5)
- moved JP3 17.1 mm to (193.3, 46.6), turned to 180 degrees
- moved C4 8.94 mm to (181.7, 53.1), turned to 180 degrees
- moved C3 7.13 mm to (181.1, 57.0), turned to 0 degrees
- moved U2 6.27 mm to (181.4, 55.1)
- moved JP1 2.78 mm to (177.7, 55.1), turned to 0 degrees
- moved Y1 0.21 mm to (191.8, 58.2)
- moved C8 0.10 mm to (192.5, 60.7)
- renumbered C17 to C16, C16 to C17
Connections:
- BT1 pad 1: VBAT -> Net-(BT1-+)
- C16 pad 1: /VDD_LDO -> Net-(JP2-A)
- C17 pad 1: /VDD_LDO -> Net-(JP3-A)
- C20 pad 1: /VDD_LDO -> /VDD_LS
- C3 pad 1: Net-(JP1-B) -> VDD
- C4 pad 1: Net-(U2-VINT) -> /VDD_LS
- JP1 pad 1: VBAT -> Net-(BT1-+)
- JP1 pad 2: Net-(JP1-B) -> VDD
- JP2 pad 1: /VDD_LDO -> Net-(JP2-A)
- JP2 pad 2: VDD -> /VDD_LS
- JP3 pad 2: VDD -> /VDD_LS
- MK1 pad 1: /VDD_LDO -> /VDD_LS
- U1 pad A3: unconnected-(U1-P1.12-PadA3) -> /UART_RX
- U1 pad B6: /BUTTON0 -> /LFCLK1
- U1 pad C3: /GPIO0 -> /LSW
- U1 pad C6: Net-(U1-P1.01) -> /LFCLK1
- U1 pad C7: unconnected-(U1-P1.02-PadC7) -> /BUTTON0
- U1 pad D5: /SCL -> unconnected-(U1-P1.03-PadD5)
- U1 pad D7: unconnected-(U1-P1.06-PadD7) -> /INT2
- U1 pad F7: /UART_RX -> /SCL
- U3 pad 10: /VDD_LDO -> Net-(JP3-A)
- U3 pad 12: /VDD_LDO -> Net-(JP2-A)
- U3 pad 6: unconnected-(U3-INT2-Pad6) -> /INT2
- Y1 pad 1: Net-(U1-P1.01) -> /LFCLK1
Routing:
- net /VDD_LDO: track 40.5 -> 0.00 mm, vias 4 -> 0
- net /VDD_LS: track 0.00 -> 20.0 mm, vias 0 -> 3
- net Net-(JP1-B): track 19.1 -> 0.00 mm, vias 2 -> 0
- net /LSW: track 0.00 -> 15.9 mm, vias 0 -> 2
- net /INT2: track 0.00 -> 13.4 mm, vias 0 -> 2
- net Net-(JP3-A): track 15.9 -> 4.26 mm, vias 2 -> 0
- net Net-(JP4-A): track 10.3 -> 0.00 mm, vias 2 -> 0
- net /GPIO0: track 5.90 -> 0.00 mm, vias 2 -> 0
- net /UART_RX: track 7.80 -> 13.6 mm, vias 2 -> 3
- net /LFCLK1: track 0.00 -> 2.77 mm, vias 0 -> 2
- net /SDA: track 27.4 -> 24.8 mm
- net Net-(U2-VINT): track 2.62 -> 0.00 mm
- net Net-(JP2-A): track 0.00 -> 2.61 mm
- net VDD: track 46.9 -> 44.7 mm, vias 7 -> 5
- net /BUTTON0: track 24.2 -> 21.9 mm
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Other:
- board text added: "H.L. A.H. M.G. G.C."
- board text removed: "LAYER 1 - 1 OZ COPPER - (0.0175 MM) LAYER 2 - PREPREG (7628, DK 4.74, 0.1855 MM) LAYER 3 - 1 OZ COPPER - (0.0350 MM) LAYER 4 - CORE (DK 4.6, 1.03 MM) LAYER 5 - 1 OZ COPPER - (0.0350 MM) LAYER 6 - PREPREG (7628, DK 4.74, 0.1855 MM) LAYER 7 - 1 OZ COPPER - (0.0175 MM)"
