File: nRF54L15_nPM2100_CR2032.kicad_sch (KiCad schematic)
At the start: 29 parts, among them Q1 Q_NMOS_GSD, SW1 SW_Push, U1 nRF54L15-CAXX, U2 nPM2100-CAXX, Y1 32.768kHz, Y2 SiT11100

Commit message: Routing complete
Parts:
- added J1: Conn_ARM_SWD_TagConnect_TC2030-NL, Connector:Tag-Connect_TC2030-IDC-NL_2x03_P1.27mm_Vertical, symbol Connector:Conn_ARM_SWD_TagConnect_TC2030-NL
- added JP1: Jumper_2_Small_Bridged, Jumper:SolderJumper-2_P1.3mm_Bridged_RoundedPad1.0x1.5mm, symbol Jumper:Jumper_2_Small_Bridged
- added R2, R3: 10kR, Resistor_SMD:R_0201_0603Metric, symbol Device:R_Small_US
- added R4: 1MR, Resistor_SMD:R_0402_1005Metric, symbol Device:R_Small_US
- added TP1, TP2: TestPoint, TestPoint:TestPoint_Pad_D1.0mm, symbol Connector:TestPoint
- AE1: footprint RF_Antenna:Johanson_2450AT18x100 -> hlord2000-RF_Antenna:Ignion_NN02-101
- C6, C9: footprint Capacitor_SMD:C_0201_0603Metric -> Capacitor_SMD:C_01005_0402Metric
- D1: value LED_Small -> APT3216LVBC/D; footprint LED_SMD:LED_0603_1608Metric -> LED_SMD:LED_1206_3216Metric
- L2, L3, L4: footprint Capacitor_SMD:C_0201_0603Metric -> Inductor_SMD:L_01005_0402Metric
- Q1: footprint (none) -> Package_TO_SOT_SMD:SOT-23
- R1: value R_Small_US -> 350R; footprint (none) -> Resistor_SMD:R_0402_1005Metric
Connections:
- net GND: now also SW1.2, U2.C2 (SYSGDEN), J1.5 (GND), R4.2; no longer AE1.1 (FEED)
- net VDD: now also J1.1 (VCC), R2.1, R3.1
- net LED: now reaches U1.B3 (P1.09)
- net LED: now also Q1.1 (G), R4.1
- net at U1.D2 (~{RESET}): now also J1.3 (~{RESET})
- net SCL: now reaches U1.D5 (P1.03)
- net SCL: now also U2.D2 (SCL), R3.2
- net SDA: now reaches U1.D6 (P1.04)
- net SDA: now also U2.D3 (SDA), R2.2
- net at U1.E3 (SWDCLK): now also J1.4 (SWCLK)
- net UART_TX: now reaches U1.E7 (P1.07)
- net UART_TX: now also TP1.1
- net at U1.F2 (SWDIO): now also J1.2 (SWDIO)
- net UART_RX: now reaches U1.F7 (P1.08)
- net UART_RX: now also TP2.1
- net at C3.1, L5.1, U2.C4 (VBAT): now also JP1.2 (B); no longer BT1.1 (+)
- net at SW1.1: now also U2.D4 (SHPHLD)
- new net: BT1.1 (+), JP1.1 (A)
- no-connect marks 1 -> 4
Other:
- moved on the sheet: BT1, SW1

Commit message: Nov. 7th 2024
Parts:
- added C14: 1nF, Capacitor_SMD:C_0201_0603Metric, symbol Device:C_Small
- added C15: 0.22uF, Capacitor_SMD:C_0201_0603Metric, symbol Device:C_Small
- added C16, C17: 100nF, Capacitor_SMD:C_0201_0603Metric, symbol Device:C_Small
- added C18: NA, Capacitor_SMD:C_0201_0603Metric, symbol Device:C_Small
- added C19, C20: 2.2uF, Capacitor_SMD:C_0201_0603Metric, symbol Device:C_Small
- added JP2: Jumper_3_Open, Jumper:SolderJumper-3_P1.3mm_Open_RoundedPad1.0x1.5mm, symbol Jumper:Jumper_3_Open
- added JP3, JP4: Jumper_2_Small_Bridged, Jumper:SolderJumper-2_P1.3mm_Bridged_RoundedPad1.0x1.5mm, symbol Jumper:Jumper_2_Small_Bridged
- added L6, L7: NA, Inductor_SMD:L_0201_0603Metric, symbol Device:L_Small
- added MK1: MP34DT05-A, hlord2000-Sensor_Audio:ST_HCLGA-4_3x4mm_P1.35mm, symbol hlord2000-Sensor_Audio:MP34DT05-A
- added U3: ADXL366, hlord2000-Sensor_Motion:Analog_LGA-12_2.20x2.30mm_P0.5mm, symbol hlord2000-Sensor_Motion:ADXL366
- AE1, U1, U2, Y2: Consigned (none) -> Y
- C10, C3: footprint Capacitor_SMD:C_0201_0603Metric -> Capacitor_SMD:C_0402_1005Metric
- C13: value 22uF -> 10uF
- C4: value 2.2uF -> 1nF
- C6, C9: footprint Capacitor_SMD:C_01005_0402Metric -> Capacitor_SMD:C_0201_0603Metric
- L2, L3, L4: footprint Inductor_SMD:L_01005_0402Metric -> Inductor_SMD:L_0201_0603Metric
- Q1: footprint Package_TO_SOT_SMD:SOT-23 -> Package_DFN_QFN:Diodes_DFN1006-3
Connections:
- net GND: now also C14.2, C15.2, C16.2, C17.2, C18.2, C19.2, C20.2, MK1.2 (SEL), MK1.5 (GND), U3.1 (SCLK), U3.11 (GND), U3.3 (MISO/ASEL), U3.7 (GND)
- net SCL: now also U3.4 (~{CS}/SCL)
- net SDA: now also U3.2 (MOSI/SDA)
- net VDD: now also JP2.2 (C), JP3.2 (B); no longer C7.1, U2.A2 (VOUT)
- net at AE1.2 (PCB_Trace): now also L7.2; no longer L4.2
- net BUTTON0: now reaches U1.B6 (P1.15)
- net BUTTON0: now also SW1.1, U2.D4 (SHPHLD)
- net GPIO0: now reaches U1.C3 (P1.10)
- net GPIO0: now also U2.C3 (GPIO0)
- net PDM_CLK: now reaches U1.E1 (P0.03)
- net PDM_CLK: now also MK1.3 (CLOCK)
- net PDM_DATA: now reaches U1.F1 (P0.01)
- net PDM_DATA: now also MK1.4 (DATA)
- net INT1: now reaches U1.G1 (P0.00)
- net INT1: now also U3.5 (INT1)
- net VBAT: now reaches BT1.1 (+), JP1.1 (A)
- net VBAT: now also JP2.3 (B)
- net at U2.A1 (VOUTLDO): now also C19.1, JP4.1 (A); no longer C4.1
- net at C3.1, JP1.2 (B), L5.1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: now also C14.1
- net at C13.1, U2.A3 (VINT): now also C4.1
- new net: C15.1, U3.9 (V_{REG_OUT})
- new net: L4.2, L6.1
- new net: C18.1, L6.2, L7.1
- new net: C7.1, JP3.1 (A), U2.A2 (VOUT)
- new net VDD_LDO: C16.1, C17.1, C20.1, JP2.1 (A), JP4.2 (B), MK1.1 (VDD), U3.10 (V_{S}), U3.12 (V_{DDIO})
- no-connect marks 4 -> 24
Other:
- moved on the sheet: AE1, BT1, C1, C10, C11, C12, C13, C2, C3, C5, C6, C7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

Commit message: Dec92024
Parts:
- removed C13: 10uF, Capacitor_SMD:C_0402_1005Metric, symbol Device:C_Small
- removed C14: 1nF, Capacitor_SMD:C_0201_0603Metric, symbol Device:C_Small
- removed C19, C7: 2.2uF, Capacitor_SMD:C_0201_0603Metric, symbol Device:C_Small
- removed JP2: Jumper_3_Open, Jumper:SolderJumper-3_P1.3mm_Open_RoundedPad1.0x1.5mm, symbol Jumper:Jumper_3_Open
- removed JP4: Jumper_2_Small_Bridged, Jumper:SolderJumper-2_P1.3mm_Bridged_RoundedPad1.0x1.5mm, symbol Jumper:Jumper_2_Small_Bridged
- removed L5: 2.2uH, Inductor_SMD:L_0402_1005Metric, symbol Device:L_Small
- removed U2: nPM2100-CAXX, nordic-lib-kicad-npm:BGA-16_4x4_1.9175x1.8975mm, symbol nordic-lib-kicad-npm:nPM2100-CAXX
- added JP2: Jumper_2_Small_Bridged, Resistor_SMD:R_0402_1005Metric, symbol Jumper:Jumper_2_Small_Bridged
- added U2: SiP32432DR3, Package_TO_SOT_SMD:SOT-363_SC-70-6, symbol Power_Management:SiP32432DR3
- C1, C2, C20: LCSC (none) -> C23630
- C10: LCSC (none) -> C15525
- C11, C16, C17, C8: LCSC (none) -> C76939
- C12: LCSC (none) -> C76941
- C15: LCSC (none) -> C701263
- C3: value 10uF -> 100nF; footprint Capacitor_SMD:C_0402_1005Metric -> Capacitor_SMD:C_0201_0603Metric; LCSC (none) -> C76939
- C4: value 1nF -> 100nF; LCSC (none) -> C76939
- C5: LCSC (none) -> C22374845
- C6, C9: LCSC (none) -> C85895
- D1: LCSC (none) -> C84273
- FB1: LCSC (none) -> C83991
- JP3: footprint Jumper:SolderJumper-2_P1.3mm_Bridged_RoundedPad1.0x1.5mm -> Resistor_SMD:R_0402_1005Metric; LCSC (none) -> C17168
- L18: renamed from C18; value NA -> 4.7nH; symbol Device:C_Small -> Device:L_Small; LCSC (none) -> C86126
- L2: LCSC (none) -> C275212
- L3: value 4.6nH -> 4.7nH; LCSC (none) -> C86126
- L4: LCSC (none) -> C307709
- L6: value NA -> 4.7nH; footprint Inductor_SMD:L_0201_0603Metric -> Capacitor_SMD:C_0201_0603Metric; LCSC (none) -> C86126
- L7: value NA -> 10nH; footprint Inductor_SMD:L_0201_0603Metric -> Capacitor_SMD:C_0201_0603Metric; LCSC (none) -> C162594
- Q1: LCSC (none) -> C7527987
- R1: value 350R -> 1kR; LCSC (none) -> C106235
- R2, R3: LCSC (none) -> C106225
- R4: LCSC (none) -> C138033
- SW1: LCSC (none) -> C127488
- U1: footprint nordic-lib-kicad-nrf54:BGA-49_7x7_2.3984x2.2309mm -> nordic-lib-kicad-nrf54:BGA-47_7x7_2.451x2.245mm
Connections:
- net BUTTON0: now also U1.C7 (P1.02); no longer U1.B6 (P1.15)
- net GND: now also U2.2 (GND), U2.5 (GND)
- net SCL: now also U1.F7 (P1.08); no longer U1.D5 (P1.03)
- net UART_RX: now also U1.A3 (P1.12); no longer U1.F7 (P1.08)
- net VDD: now also C3.1, JP1.2 (B), U2.4 (IN); no longer JP3.2 (B)
- net INT2: now reaches U3.6 (INT2)
- net INT2: now also U1.D7 (P1.06)
- net LFCLK1: now reaches U1.C6 (P1.01), Y1.1
- net LFCLK1: now also U1.B6 (P1.15)
- net at JP3.1 (A): now also C17.1, U3.10 (V_{S})
- net VDD_LS: now reaches C4.1
- net VDD_LS: now also C20.1, JP3.2 (B), MK1.1 (VDD), JP2.2 (B), U2.1 (OUT)
- net GPIO0 renamed LSW
- net LSW: now also U2.3 (~{ON})
- net VBAT: no longer names the net of BT1.1 (+), JP1.1 (A)
- removed net VDD_LDO: C16.1, C17.1, C20.1, MK1.1 (VDD), U3.10 (V_{S}), U3.12 (V_{DDIO})
- new net: C16.1, JP2.1 (A), U3.12 (V_{DDIO})
- no-connect marks 24 -> 18
Other:
- moved on the sheet: C15, C16, C17, D1, Q1, R1, R2, R3, R4, SW1, TP2, U3

Commit message: Updated for production
Parts:
- BT1: footprint Battery:BatteryHolder_Multicomp_BC-2001_1x2032 -> nRF54L15_Battery:BatteryHolder_Multicomp_BC-2001_1x2032; PartId (none) -> 100500047
- C1, C2, C20: PartId (none) -> 100200660
- C10: PartId (none) -> 100200383
- C11, C16, C17, C3, C4, C8: PartId (none) -> 100200469
- C12: PartId (none) -> 100200491
- C15: PartId (none) -> 100200487
- C5: PartId (none) -> 100200092
- C6, C9: PartId (none) -> 100200086
- D1: value APT3216LVBC/D -> LB Q39E; footprint LED_SMD:LED_1206_3216Metric -> LED_SMD:LED_0603_1608Metric; PartId (none) -> 101400142
- FB1: PartId (none) -> 100300419
- J1: now not fitted
- JP1, TP1, TP2: now not fitted; now left out of the parts list
- JP2, JP3: PartId (none) -> 100100109
- L1: PartId (none) -> 100300441
- L18, L3: PartId (none) -> 100300231
- L2: PartId (none) -> 100300223
- L4: PartId (none) -> 100300016
- L6: value 4.7nH -> 4.9nH; PartId (none) -> 100300233
- L7: PartId (none) -> 100300242
- Q1: PartId (none) -> 101300187
- R1: PartId (none) -> 100100171
- R2, R3: PartId (none) -> 100100065
- R4: PartId (none) -> 100100265
- SW1: PartId (none) -> 101500104
- U1: PartId (none) -> 102000283
Other:
- title: (none) -> nRF54L Tiny Board

Commit message: Fixed issues w/ mousebites, added stitching vias, added fiducials
Parts:
- added FID1, FID2, FID3: Fiducial, Fiducial:Fiducial_0.5mm_Mask1mm, symbol Mechanical:Fiducial
- AE1: PartId (none) -> 100700079; Ship from Helmut (none) -> Y/optional
- MK1: PartId (none) -> MP34DT05-A
- U2: PartId (none) -> SiP32432DR3
- U3: PartId (none) -> ADXL366; Ship from Helmut (none) -> Y
- Y1: PartId (none) -> ECS-.327-9-1210-TR
- Y2: PartId (none) -> SiT11100; Ship from Helmut (none) -> Y
